File: Hardware/NO_Sensor_Breakout.sch (KiCad schematic (older format))
At the start: 5 parts

Commit message: Finished BOM
Parts:
- C1: renamed from C?; footprint (none) -> Capacitor_SMD:C_0603_1608Metric_Pad1.08x0.95mm_HandSolder
- Conn1: renamed from Conn?; footprint (none) -> MRDT_Connectors:MOLEX_SL_04_Vertical
- R1, R2: renamed from R?; footprint (none) -> Resistor_SMD:R_0603_1608Metric_Pad0.98x0.95mm_HandSolder
- gave numbers to parts that had none: 1
Changed lines of the file:
@@
 $EndDescr
 $Comp
-L MRDT_Connectors:Molex_SL_04 Conn?
+L MRDT_Connectors:Molex_SL_04 Conn1
 U 1 1 5FD004AF
 P 4120 2550
-F 0 "Conn?" H 4062 2363 60  0000 C CNN
+F 0 "Conn1" H 4062 2363 60  0000 C CNN
 F 1 "Molex_SL_04" H 4062 2469 60  0000 C CNN
-F 2 "" H 4120 2550 60  0001 C CNN
+F 2 "MRDT_Connectors:MOLEX_SL_04_Vertical" H 4120 2550 60  0001 C CNN
 F 3 "" H 4120 2550 60  0001 C CNN
 	1    4120 2550
@@
 $EndComp
 $Comp
-L power:GND #PWR?
+L power:GND #PWR0101
 U 1 1 5FD00E95
 P 5700 3800
-F 0 "#PWR?" H 5700 3550 50  0001 C CNN
+F 0 "#PWR0101" H 5700 3550 50  0001 C CNN
 F 1 "GND" H 5705 3627 50  0000 C CNN
 F 2 "" H 5700 3800 50  0001 C CNN
@@
 NoConn ~ 5750 2700
 $Comp
-L Device:C_Small C?
+L Device:C_Small C1
 U 1 1 5FD035DE
 P 4990 3150
-F 0 "C?" H 4770 3220 50  0000 L CNN
+F 0 "C1" H 4770 3220 50  0000 L CNN
 F 1 "10uF" H 4730 3150 50  0000 L CNN
-F 2 "" H 4990 3150 50  0001 C CNN
+F 2 "Capacitor_SMD:C_0603_1608Metric_Pad1.08x0.95mm_HandSolder" H 4990 3150 50  0001 C CNN
 F 3 "~" H 4990 3150 50  0001 C CNN
 	1    4990 3150
@@
 	4990 3000 4990 3050
 $Comp
-L power:GND #PWR?
+L power:GND #PWR0102
 U 1 1 5FD045BE
 P 4990 3290
-F 0 "#PWR?" H 4990 3040 50  0001 C CNN
+F 0 "#PWR0102" H 4990 3040 50  0001 C CNN
 F 1 "GND" H 4990 3150 50  0000 C CNN
 F 2 "" H 4990 3290 50  0001 C CNN
@@
 	4990 3250 4990 3290
 $Comp
-L power:+3.3V #PWR?
+L power:+3.3V #PWR0103
 U 1 1 5FD05EF3
 P 4740 2170
-F 0 "#PWR?" H 4740 2020 50  0001 C CNN
+F 0 "#PWR0103" H 4740 2020 50  0001 C CNN
 F 1 "+3.3V" H 4620 2280 50  0000 C CNN
 F 2 "" H 4740 2170 50  0001 C CNN
@@
 	4460 2800 4460 2960
 $Comp
-L power:GND #PWR?
+L power:GND #PWR0104
 U 1 1 5FD0761E
 P 4460 2960
-F 0 "#PWR?" H 4460 2710 50  0001 C CNN
+F 0 "#PWR0104" H 4460 2710 50  0001 C CNN
 F 1 "GND" H 4460 2830 50  0000 C CNN
 F 2 "" H 4460 2960 50  0001 C CNN
@@
 	5600 2600 5600 2700
 $Comp
-L Device:R R?
+L Device:R R1
 U 1 1 5FD24A0B
 P 5450 2420
-F 0 "R?" H 5300 2420 50  0000 L CNN
+F 0 "R1" H 5300 2420 50  0000 L CNN
 F 1 "1K" V 5450 2380 50  0000 L CNN
-F 2 "" V 5380 2420 50  0001 C CNN
+F 2 "Resistor_SMD:R_0603_1608Metric_Pad0.98x0.95mm_HandSolder" V 5380 2420 50  0001 C CNN
 F 3 "~" H 5450 2420 50  0001 C CNN
 	1    5450 2420
@@
 $EndComp
 $Comp
-L Device:R R?
+L Device:R R2
 U 1 1 5FD24F74
 P 5600 2420
-F 0 "R?" H 5660 2420 50  0000 L CNN
+F 0 "R2" H 5660 2420 50  0000 L CNN
 F 1 "1K" V 5600 2380 50  0000 L CNN
-F 2 "" V 5530 2420 50  0001 C CNN
+F 2 "Resistor_SMD:R_0603_1608Metric_Pad0.98x0.95mm_HandSolder" V 5530 2420 50  0001 C CNN
 F 3 "~" H 5600 2420 50  0001 C CNN
 	1    5600 2420
@@
 	5450 2210 4740 2210
 $Comp
-L MRDT_ICs:USEQGSEAN8L180 U?
+L MRDT_ICs:USEQGSEAN8L180 U1
 U 1 1 5FCFEE7F
 P 5500 2800
-F 0 "U?" H 5645 2520 50  0000 L CNN
+F 0 "U1" H 5645 2520 50  0000 L CNN
 F 1 "USEQGSEAN8L180" H 5360 2455 50  0000 L CNN
 F 2 "MRDT_ICs:USEQGSEAN8L180" H 5500 2700 50  0001 C CNN
